File: hw/project.sch (KiCad schematic (older format))
At the start: 42 parts, among them P1 Inputs, P10 Tank2High, P2 Serial, P3 DS18B20, P4 DS18B20, P5 I2C, P6 I2C, P7 Milone eTape Sensor, P8 LowWater, P9 Tank1High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

Commit message: removed some un-needed components, updated faulty modules and reduced board size.
Parts:
- removed C6: 0.1uF, symbol C
- removed D5: WaterLevel_Calibrate_LED, symbol LED
- removed D6: PH_Calibrate_LED, symbol LED
- removed D7: Replace_PH_LED, symbol LED
- removed D8: Bad_Water_LED, symbol LED
- removed P2: Serial, symbol CONN_6
- removed R10, R11, R12, R9: 560, symbol R
- removed SW2: Select, symbol SW_PUSH
- removed U3: 74HC595, symbol 74HC595
- D1: value Good_PH_LED -> LED
- D2: value Good_Water_LED -> LED
- D3: value High_LED -> LED
- D4: value Low_LED -> LED
- SW1: value Function -> Pump
- SW3: value Special -> Light
Connections:
- net labels added: Error_LED, Light_Switch, Link_LED, Pump_Switch
- net labels removed: Clock, Data, Function_Switch, HighCalibrate, Latch, LowCalibrate, PHCalibrate, RX, ReplacePHProbe, Reset, Select_Switch, Special_Switch, TX, WaterCalibrate
- wire segments 176 -> 121
- no-connect marks 2 -> 4
Other:
- note added: "Light Toggle"
- note added: "Water Toggle\n"
- note removed: "Light Toggle / Select"
- note removed: "Serial Adaptor Connector"
- note removed: "Shift Register"
- note removed: "Water Toggle / Function"
- moved on the sheet: C2, C3, C4, C5, P10, P5, P6, P7, P8, P9, R3, R4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
