File: hw/Hydroponics_Controller.kicad_pcb (KiCad board)
At the start: 2 copper layers, 55 x 46 mm, 35 parts, among them K1 1Wire, K2 1Wire, P1 I2C, P2 I2C, P3 Relay, P4 Low Water, P5 Tank 1 High, P6 Tank 2 High, P7 eTape, P8 Power In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

Commit message: Added RTC to board. Corrected error using A6/A7 as digital pins...
Parts:
- added BT1: BATTERY, 10to7_discrete:CRC2032, B.Cu at (225.5, 97.7)
- added C6: 0.1uF, 10to7_sm_standard:SM0402, F.Cu at (231.3, 103.2)
- added R10: 10k, 10to7_sm_standard:SM0402, F.Cu at (232.5, 105.2)
- added R9: 10k, 10to7_sm_standard:SM0402, F.Cu at (231.3, 105.2)
- added U3: DS3231, SMD_Packages:SO16W, F.Cu at (224.3, 101.2)
- P4: value Low Water -> LowWater
- P5: value Tank 1 High -> Tank1High
- P6: value Tank 2 High -> Tank2High
- P8: value Power In -> Power_In
- R3, R4: value 4k7 -> 10k
- moved SW_Light1 23.0 mm to (229.8, 120.7), turned to 180 degrees
- moved 3mmHole_2 17.6 mm to (237.7, 83.7)
- moved 3mmHole_3 17.6 mm to (237.7, 121.7)
- moved D1 17.6 mm to (238.8, 92.2)
- moved D2 17.6 mm to (233.5, 92.2)
- moved D3 17.6 mm to (238.8, 102.7)
- moved D4 17.6 mm to (238.8, 113.2)
- moved R1 17.6 mm to (238.8, 89.2)
- moved R2 17.6 mm to (233.5, 89.2)
- moved R5 17.6 mm to (238.8, 99.7)
- moved R6 17.6 mm to (238.8, 110.2)
- moved SW_Pump1 8.61 mm to (219.5, 120.7), turned to 180 degrees
- moved 3mmHole_1 2.58 mm to (175.7, 83.7)
- moved 3mmHole_4 2.58 mm to (175.7, 121.7)
- moved C1 2.58 mm to (192.4, 87.9)
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Connections:
- U2 pad 19: /WaterDepth -> /Pump_Switch
- U2 pad 20: /WaterDepthRef -> /Link_LED
- U2 pad 25: /Pump_Switch -> /WaterDepth
- U2 pad 26: /Link_LED -> /WaterDepthRef
Routing:
- net GND: track 68.0 -> 220.9 mm
- net Net-(BT1-Pad1): track 0.00 -> 26.5 mm, vias 0 -> 1
- net +5V: track 116.6 -> 131.8 mm
- net /Error_LED: track 8.02 -> 22.6 mm
- net /Light_Switch: track 34.4 -> 48.7 mm
- net /PumpRelay: track 35.8 -> 48.9 mm
- net /WaterDepthRef: track 6.43 -> 19.2 mm
- net VCC: track 51.9 -> 64.4 mm
- net /Pump_Switch: track 33.1 -> 44.9 mm
- net /WaterDepth: track 10.9 -> 22.5 mm
- net /SCL: track 12.2 -> 23.6 mm
- net /LightRelay: track 38.1 -> 49.5 mm
- net /SDA: track 12.6 -> 20.4 mm
- net /Link_LED: track 40.1 -> 45.9 mm
- net Net-(R9-Pad2): track 0.00 -> 5.78 mm
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Other:
- board size 55 x 46 mm -> 70 x 46 mm
- net class Default: clearance 0 -> 0.2
- rule trace_clearance: 0 -> 0.2
- board text added: "10to7.com Hydroponics Controller Version 0.06"
- board text added: "A0"
- board text added: "A1"
- board text added: "D4 D5 A7 A6 D3"
- board text added: "D6 A0 D7 A5 D8 A1"
- board text removed: "10to7.com Hydroponics Controller Version 0.05"
- board text removed: "A6"
- board text removed: "A7"
- board text removed: "D4 D5 A1 A0 D3"
- board text removed: "D6 A6 D7 A5 D8 A7"

Commit message: Fixed the missing pullup resistor from the 1 wire connector
Parts:
- added R11: 4K7, 10to7_sm_standard:SM0402, F.Cu at (203.8, 115.7)
Routing:
- net GND: track 220.9 -> 211.1 mm
- net /1Wire: track 14.4 -> 16.9 mm
- net +5V: track 131.8 -> 134.2 mm
Other:
- board text added: "10to7.com Hydroponics Controller Version 0.07"
- board text removed: "10to7.com Hydroponics Controller Version 0.06"
- board text removed: "D8"

Commit message: updated to fix I2C connected to wrong pins. Also changed cap to 0402
Parts:
- C1: footprint 10to7_sm_standard:SM0603 -> 10to7_sm_standard:SM0402
- moved D4 18.8 mm to (220.1, 115.5), turned to 0 degrees
- moved R5 16.7 mm to (233.6, 115.5), turned to 0 degrees
- moved R6 16.5 mm to (223.1, 115.5), turned to 0 degrees
- moved D3 15.2 mm to (230.6, 115.5), turned to 0 degrees
- moved C1 1.10 mm to (193.4, 88.5)
- moved C4 0.77 mm to (193.4, 89.8)
- moved C5 0.57 mm to (193.3, 119.2)
- moved P8 0.57 mm to (186.5, 120.2)
- moved R11 0.57 mm to (204.3, 116.0)
- moved U2 0.57 mm to (197.0, 104.1)
- moved D1 0.57 mm to (239.3, 92.4)
- moved D2 0.57 mm to (234.0, 92.4)
- moved R1 0.57 mm to (239.3, 89.4)
- moved R2 0.57 mm to (234.0, 89.4)
- moved BT1 0.57 mm to (226.0, 97.9)
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Connections:
- U2 pad 1: (no net) -> Net-(U2-Pad1)
- U2 pad 2: (no net) -> Net-(U2-Pad2)
- U2 pad 23: /LowWater -> /SDA
- U2 pad 24: /Light_Switch -> /SCL
- U2 pad 28: (no net) -> Net-(U2-Pad28)
- U2 pad 3: (no net) -> Net-(U2-Pad3)
- U2 pad 7: /SDA -> Net-(U2-Pad7)
- U2 pad 8: /SCL -> Net-(U2-Pad8)
- U3 pad 4: (no net) -> Net-(U3-Pad4)
Routing:
- net /Light_Switch: track 48.7 -> 7.60 mm
- net /LowWater: track 21.1 -> 0.00 mm
- net /SDA: track 20.4 -> 37.0 mm
- net GND: track 211.1 -> 227.0 mm
- net /PumpRelay: track 48.9 -> 38.6 mm
- net /Pump_Switch: track 44.9 -> 53.9 mm
- net /LightRelay: track 49.5 -> 41.4 mm
- net VCC: track 64.4 -> 56.4 mm
- net /MOSI: track 27.8 -> 33.6 mm
- net /WaterDepth: track 22.5 -> 19.0 mm
- net /IRQ: track 47.9 -> 51.3 mm
- net +5V: track 134.2 -> 137.1 mm
- net /SCL: track 23.6 -> 26.1 mm
- net /WaterDepthRef: track 19.2 -> 20.7 mm
- net Net-(BT1-Pad1): track 26.5 -> 25.2 mm
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Other:
- board text added: "10to7.com Hydroponics Controller Version 0.08"
- board text added: "A4 A5 A7 A6 D3"
- board text added: "D4"
- board text added: "D6 A0 D7 D5 D8 A1"
- board text removed: "10to7.com Hydroponics Controller Version 0.07"
- board text removed: "A4"
- board text removed: "D4 D5 A7 A6 D3"
- board text removed: "D6 A0 D7 A5 D8 A1"
